File: RFXCOM.kicad_pcb (KiCad board)
At the start: 2 copper layers, 23 x 45.8 mm, 9 parts, among them J1 Conn_Coaxial, J2 Conn_Coaxial, J3 Conn_01x01, J4 Rx, J5 Tx, U1 arduino_mega_pro_embedded

Commit message: stm32 based pcb
Parts:
- added C10: 1u, Capacitor_SMD:C_0603_1608Metric_Pad1.08x0.95mm_HandSolder, F.Cu at (134.0, 97.4)
- added C11: 10n, Capacitor_SMD:C_0603_1608Metric_Pad1.08x0.95mm_HandSolder, F.Cu at (136.2, 97.4)
- added C12: 2u, Capacitor_SMD:C_0805_2012Metric_Pad1.18x1.45mm_HandSolder, F.Cu at (112.9, 89.8)
- added C13: 3u3, Capacitor_SMD:C_0805_2012Metric_Pad1.18x1.45mm_HandSolder, F.Cu at (105.7, 89.8)
- added C14: 1u, Capacitor_SMD:C_0805_2012Metric_Pad1.18x1.45mm_HandSolder, F.Cu at (103.0, 89.8)
- added C4: 4u7, Capacitor_SMD:C_0805_2012Metric_Pad1.18x1.45mm_HandSolder, F.Cu at (135.2, 89.8)
- added C5: 10p, Capacitor_SMD:C_0603_1608Metric_Pad1.08x0.95mm_HandSolder, F.Cu at (130.6, 91.0)
- added C6: 10p, Capacitor_SMD:C_0603_1608Metric_Pad1.08x0.95mm_HandSolder, F.Cu at (130.6, 97.0)
- added C7: 100n, Capacitor_SMD:C_0603_1608Metric_Pad1.08x0.95mm_HandSolder, F.Cu at (136.8, 91.4)
- added C8: 100n, Capacitor_SMD:C_0603_1608Metric_Pad1.08x0.95mm_HandSolder, F.Cu at (132.0, 101.0)
- added C9: 100n, Capacitor_SMD:C_0603_1608Metric_Pad1.08x0.95mm_HandSolder, F.Cu at (144.2, 99.0)
- added D1: LED_AGRB, LED_SMD:LED_RGB_Wuerth-PLCC4_3.2x2.8mm_150141M173100, F.Cu at (110.8, 99.8)
- added D2: ESD9X5.0ST5G, Diode_SMD:D_SOD-923, F.Cu at (55.8, 44.5)
- added FB1: 120R, Inductor_SMD:L_1206_3216Metric_Pad1.22x1.90mm_HandSolder, F.Cu at (100.4, 89.0)
- added J6: USB_C_Receptacle_USB2.0, Connector_USB:USB_C_Receptacle_HRO_TYPE-C-31-M-12, F.Cu at (49.0, 47.5)
- added J7: SWD, Connector_PinHeader_1.27mm:PinHeader_2x03_P1.27mm_Vertical_SMD, F.Cu at (143.6, 88.0)
- added R1: 5k1, Resistor_SMD:R_0805_2012Metric_Pad1.20x1.40mm_HandSolder, F.Cu at (100.8, 99.4)
- added R2: 5k1, Resistor_SMD:R_0805_2012Metric_Pad1.20x1.40mm_HandSolder, F.Cu at (100.4, 95.2)
- added R3: 130, Resistor_SMD:R_0805_2012Metric_Pad1.20x1.40mm_HandSolder, F.Cu at (113.2, 96.0)
- added R4: 30, Resistor_SMD:R_0805_2012Metric_Pad1.20x1.40mm_HandSolder, F.Cu at (108.4, 96.0)
- added R5: 30, Resistor_SMD:R_0805_2012Metric_Pad1.20x1.40mm_HandSolder, F.Cu at (110.8, 96.0)
- added U2: USBLC6-2SC6, Package_TO_SOT_SMD:SOT-23-6, F.Cu at (58.4, 47.0)
- added U3: LD2981ABU33TR, Package_TO_SOT_SMD:SOT-89-3, F.Cu at (109.3, 89.2)
- added Y1: 16M, Crystal:Crystal_SMD_Abracon_ABM8G-4Pin_3.2x2.5mm, F.Cu at (130.6, 94.0)
- J1: value Conn_Coaxial -> TX Antenna
- J2: value Conn_Coaxial -> RX Antenna
- J3: value Conn_01x01 -> SWD_Connector; footprint Connector_PinHeader_2.54mm:PinHeader_1x01_P2.54mm_Vertical -> Connector_PinHeader_2.54mm:PinHeader_1x06_P2.54mm_Vertical
- J5: footprint Connector_PinHeader_2.54mm:PinHeader_1x03_P2.54mm_Vertical -> Connector_PinHeader_2.54mm:PinHeader_1x04_P2.54mm_Vertical
- U1: value arduino_mega_pro_embedded -> STM32L412KBTx; footprint rf_components:arduino_mega_pro_embedded -> Package_DFN_QFN:QFN-32-1EP_5x5mm_P0.5mm_EP3.45x3.45mm
- moved J2 81.4 mm to (53.0, 30.0), turned to -90 degrees
- moved J5 56.0 mm to (72.0, 26.9), turned to 0 degrees
- moved J3 54.7 mm to (163.0, 84.2), turned to 0 degrees
- moved C3 45.1 mm to (80.2, 36.2), turned to 90 degrees
- moved C2 42.2 mm to (82.4, 36.2), turned to 90 degrees
- moved U1 40.2 mm to (140.6, 95.2), turned to 0 degrees
- moved J1 39.7 mm to (82.6, 30.0), turned to -90 degrees
- moved C1 39.2 mm to (84.6, 36.2), turned to 90 degrees
- moved J4 37.2 mm to (87.8, 39.4), turned to -90 degrees
Connections:
- J1 pad 1: Net-(J3-Pad1) -> Net-(J1-Pad1)
- J3 pad 1: Net-(J3-Pad1) -> unconnected-(J3-Pad1)
- J5 pad 1: GND -> Net-(J1-Pad1)
- J5 pad 2: +5V -> GND
- J5 pad 3: /Tx_DATA -> +5V
Routing:
- net GND: track 5.20 -> 46.1 mm, vias 4 -> 9
- net +5V: track 51.1 -> 77.5 mm, vias 1 -> 2
- net +3.3V: track 0.00 -> 19.7 mm, vias 0 -> 2
- net Net-(J1-Pad1): track 0.00 -> 11.5 mm
- net /Rx_DATA: track 9.32 -> 0.00 mm
- net Net-(J3-Pad1): track 7.04 -> 0.00 mm
- net /USB & Power Supply/USB_C_D-: track 0.00 -> 6.37 mm
- net /USB & Power Supply/USB_C_D+: track 0.00 -> 6.34 mm
- net Net-(C5-Pad2): track 0.00 -> 5.55 mm
- net Net-(D1-Pad3): track 0.00 -> 3.43 mm
- net Net-(D1-Pad4): track 0.00 -> 3.31 mm
- net +3.3VA: track 0.00 -> 3.27 mm, vias 0 -> 1
- net unconnected-(U1-PadVIN_1): track 2.54 -> 0.00 mm
- net +3V3: track 2.54 -> 0.00 mm
- net Net-(D1-Pad2): track 0.00 -> 2.31 mm
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Other:
- board size 23 x 45.8 mm -> 101 x 77 mm
